File: EEPROM ONLY memory board.brd (EAGLE design)
At the start: 102.5 x 49.5 mm, 53 parts, among them IC1 28C64AVS, IC4 74AC590D, IC5 74AC590D, J2 AVR_SPI_PROG_3X2SMD, U4 ATMEGA328P_TQFP, Y2 16MHz

Commit message: Add files via upload
Parts:
- removed R11: 10K, adafruit:R1206
- added R32, R34: JMP, adafruit:R1206
- added R33: 470ohm, adafruit:R1206
- added RX2, RX3, RX4, RX5, RX6, RX7, RX8, RX9: (no value), SparkFun-Connectors:PAD.03X.03
- moved R20 3.42 mm to (42.8, 44.3)
- moved R7 2.54 mm to (30.7, 28.7)
- moved R25 1.15 mm to (36.8, 29.6)
- moved R5 0.90 mm to (33.0, 28.7)
- moved Y2 0.63 mm to (24.4, 33.0)
- moved R10 0.51 mm to (52.1, 34.8)
- moved R8 0.51 mm to (51.6, 41.9)
- moved R22 0.51 mm to (39.1, 36.1)
- moved D2 0.38 mm to (34.3, 41.1)
Connections:
- new net N$17: R33.2, X1.3
- new net N$19: R33.1, RX7.P$1
- net A0: now also RX5.P$1
- net A8: now also RX6.P$1
- net COUNTER_CLK: now also RX3.P$1
- net EEP_!OE: now also RX2.P$1
- net EEP_!WE: now also RX4.P$1
- net GND: now also R32.1, R32.2; no longer R11.2
- net N$12: now also R34.1, R34.2
- net N$6: no longer R11.1
- net VGA_1: now also RX8.P$1
- net VGA_2: now also RX9.P$1
Routing:
- net GND: track 392.7 -> 433.6 mm
- net N$12: track 34.3 -> 65.5 mm
- net N$6: track 2.98 -> 20.0 mm
- net N$17: track 0.00 -> 6.26 mm
- net EEP_!WE: track 69.5 -> 72.9 mm
- net EEP_!OE: track 84.9 -> 86.4 mm
- net A0: track 50.6 -> 52.0 mm
- net A8: track 16.4 -> 17.6 mm
- net VCC: track 333.0 -> 334.1 mm
- net N$2: track 5.02 -> 6.07 mm
- net N$4: track 27.4 -> 28.3 mm
- net VGA_2: track 12.5 -> 11.7 mm
- net RST: track 51.5 -> 52.2 mm
- net COUNTER_CLK: track 68.2 -> 68.8 mm
- net N$11: track 3.18 -> 3.69 mm
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Other:
- board text added: "!OE"
- board text added: "!WE"
- board text added: "A0"
- board text added: "A8"
- board text added: "ADC"
- board text added: "I/O 0"
- board text added: "I/O 7"
