File: EEPROM ONLY memory board.sch (EAGLE design)
At the start: 53 parts, among them IC1 28C64AVS, IC4 74AC590D, IC5 74AC590D, J2 AVR_SPI_PROG_3X2SMD, U4 ATMEGA328P_TQFP, Y2 16MHz

Commit message: Add files via upload
Parts:
- removed R11: 10K, adafruit:R-US_R1206
- added R32, R34: JMP, adafruit:R-US_R1206
- added R33: 470ohm, adafruit:R-US_R1206
- added RX2, RX3, RX4, RX5, RX6, RX7, RX8, RX9: TEST-POINT3, SparkFun-Connectors:TEST-POINT3
Connections:
- new net N$17: R33.2, X1.3
- new net N$19: R33.1, RX7.1
- net A0: now also RX5.1
- net A8: now also RX6.1
- net COUNTER_CLK: now also RX3.1
- net EEP_!OE: now also RX2.1
- net EEP_!WE: now also RX4.1
- net GND: now also R32.1, R32.2; no longer R11.2
- net N$12: now also R34.1, R34.2
- net N$6: no longer R11.1
- net VGA_1: now also RX8.1
- net VGA_2: now also RX9.1
